File: Optinal Balanced Driver Board/Source/BalancedDriverBoard.sch (KiCad schematic (older format))
At the start: 132 parts, among them J1 B3B-EH, J10 PinHeader_01x02, J11 PinHeader_01x02, J2 B3B-EH, J3 PD3MRMS2, J4 PD3MRMS2, J5 PD3MRMS2, J6 PD3MRMS2, J7 Conn_01x03, J8 PinHeader_01x02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

Commit message: Fixed U1 - U4 parts number as OPA1632.
Parts:
- C10, C11, C12, C39, C42, C9: JLPCB# (none) -> C15850
- C13, C14, C15, C16, C37, C40, C44: JLPCB# (none) -> C49678
- C17, C18, C19, C20, C21, C22, C23, C24, C25, C26, C27, C28: JLPCB# (none) -> C1790
- C38: JLPCB# (none) -> C28323
- D1, D2, D3: value LED_GRN -> LED_RED; JLPCB# (none) -> C2286
- Q1, Q2, Q3, Q4, Q5, Q6, Q7, Q8: JLPCB# (none) -> C79973
- R1, R2, R3, R4, R5, R6, R7, R8: JLPCB# (none) -> C17414
- R10, R12, R14, R16: JLPCB# (none) -> C4328
- R11, R13, R15, R9: JLPCB# (none) -> C17673
- R17, R18, R19, R20, R21, R22, R23, R24: JLPCB# (none) -> C17782
- R25, R26, R27, R28, R29, R30, R31, R32: JLPCB# (none) -> C17560
- R33, R34, R35, R36, R37, R38, R39, R40: JLPCB# (none) -> C17798
- R41, R42, R43, R44, R45, R46, R47, R48, R50, R51: JLPCB# (none) -> C17713
- R49: JLPCB# (none) -> C17513
- R52, R53, R54, R55: JLPCB# (none) -> C17561
- U1, U2, U3, U4: value OPA1611 -> OPA1632; JLPCB# (none) -> C86715
- U5: JLPCB# (none) -> C86723
